Commit message: Added EKF

File: external/turtlebot3_description/urdf/turtlebot3_burger.gazebo.xacro (robot description, xacro)
@@ -119,6 +119,6 @@
       </ray>
       <plugin name="gazebo_ros_lds_lfcd_controller" filename="libgazebo_ros_laser.so">
-        <topicName>scan</topicName>
-        <frameName>base_scan</frameName>
+        <topicName>/laser/scan</topicName>
+        <frameName>map</frameName>
       </plugin>
     </sensor>

File: external/turtlebot3_description/urdf/turtlebot3_burger.urdf.xacro (robot description, xacro)
@@ -53,8 +53,8 @@
     <inertial>
       <origin xyz="0 0 0" />
-      <mass value="2.8498940e-02" />
-      <inertia ixx="1.1175580e-05" ixy="-4.2369783e-11" ixz="-5.9381719e-09"
-               iyy="1.1192413e-05" iyz="-1.4400107e-11"
-               izz="2.0712558e-05" />
+      <mass value="2.8498940e-01" />
+      <inertia ixx="1.1175580e-03" ixy="-4.2369783e-9" ixz="-5.9381719e-07"
+               iyy="1.1192413e-03" iyz="-1.4400107e-9"
+               izz="2.0712558e-03" />
       </inertial>
   </link>
@@ -81,8 +81,8 @@
     <inertial>
       <origin xyz="0 0 0" />
-      <mass value="2.8498940e-02" />
-      <inertia ixx="1.1175580e-05" ixy="-4.2369783e-11" ixz="-5.9381719e-09"
-               iyy="1.1192413e-05" iyz="-1.4400107e-11"
-               izz="2.0712558e-05" />
+      <mass value="2.8498940e-01" />
+      <inertia ixx="1.1175580e-03" ixy="-4.2369783e-9" ixz="-5.9381719e-07"
+               iyy="1.1192413e-03" iyz="-1.4400107e-9"
+               izz="2.0712558e-03" />
       </inertial>
   </link>
